Commit message: four wheel control

File: example_control_file/epmc_ros2_control.xacro (robot description, xacro)
@@ -5,22 +5,40 @@
       <hardware>
         <plugin>epmc_v2_ros_hw_plugin/EPMC_V2_HardwareInterface</plugin>
-        <param name="motor0_wheel_name">left_wheel_joint</param>
-        <param name="motor1_wheel_name">right_wheel_joint</param>
+        <param name="motor0_wheel_name">front_left_wheel_joint</param>
+        <param name="motor1_wheel_name">front_right_wheel_joint</param>
+        <param name="motor2_wheel_name">rear_left_wheel_joint</param>
+        <param name="motor3_wheel_name">rear_right_wheel_joint</param>
         <param name="port">/dev/ttyUSB0</param>
         <!-- <param name="port">/dev/serial/by-path/pci-0000:00:14.0-usb-0:1.4:1.0-port0</param> -->
         <param name="cmd_vel_timeout_ms">2000</param>
       </hardware>
-      <joint name="left_wheel_joint">
+      <joint name="front_left_wheel_joint">
         <command_interface name="velocity">
-            <param name="min">-10.0</param> <!-- rad/sec -->
-            <param name="max">10.0</param> <!-- rad/sec -->
+            <param name="min">-8.0</param>
+            <param name="max">8.0</param>
         </command_interface>
         <state_interface name="position"/>
         <state_interface name="velocity"/>
       </joint>
-      <joint name="right_wheel_joint">
+      <joint name="front_right_wheel_joint">
         <command_interface name="velocity">
-            <param name="min">-10.0</param> <!-- rad/sec -->
-            <param name="max">10.0</param> <!-- rad/sec -->
+            <param name="min">-8.0</param>
+            <param name="max">8.0</param>
+        </command_interface>
+        <state_interface name="position"/>
+        <state_interface name="velocity"/>
+      </joint>
+      <joint name="rear_left_wheel_joint">
+        <command_interface name="velocity">
+            <param name="min">-8.0</param>
+            <param name="max">8.0</param>
+        </command_interface>
+        <state_interface name="position"/>
+        <state_interface name="velocity"/>
+      </joint>
+      <joint name="rear_right_wheel_joint">
+        <command_interface name="velocity">
+            <param name="min">-8.0</param>
+            <param name="max">8.0</param>
         </command_interface>
         <state_interface name="position"/>
